File: INDY THE TREASURE HUNTER/INDY THE TREASURE HUNTER.kicad_sch (KiCad schematic)
At the start: 3 parts

Commit message: .
Parts:
- removed U? (x2): BOB-12009, CONV_BOB-12009, symbol BOB-12009:BOB-12009
- removed U?: ARDUINO UNO, MODULE_ABX00027, symbol ARDUINO UNO:ABX00027
Other:
- added sheet MICROCONTROLLER (MICROCONTROLLER.kicad_sch)
Changed lines of the file:
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@@
 (kicad_sch (version 20230121) (generator eeschema)
   (paper "A4")
-  (symbol (lib_name "BOB-12009_1") (lib_id "BOB-12009:BOB-12009") (at 43.18 99.06 0) (unit 1)
-    (in_bom yes) (on_board yes) (dnp no) (fields_autoplaced)
-    (property "Reference" "U?" (at 43.18 85.09 0)
-      (effects (font (size 1.27 1.27)))
-    )
-    (property "Value" "BOB-12009" (at 43.18 87.63 0)
-      (effects (font (size 1.27 1.27)))
-    )
-    (property "Footprint" "CONV_BOB-12009" (at 43.18 99.06 0)
-      (effects (font (size 1.27 1.27)) (justify bottom) hide)
-    )
-    (property "Datasheet" "" (at 43.18 99.06 0)
-      (effects (font (size 1.27 1.27)) hide)
-    )
-    (property "DigiKey_Part_Number" "1568-1209-ND" (at 43.18 99.06 0)
-      (effects (font (size 1.27 1.27)) (justify bottom) hide)
-    )
-    (property "MF" "SparkFun" (at 43.18 99.06 0)
-      (effects (font (size 1.27 1.27)) (justify bottom) hide)
-    )
-    (property "MAXIMUM_PACKAGE_HEIGHT" "N/A" (at 43.18 99.06 0)
-      (effects (font (size 1.27 1.27)) (justify bottom) hide)
-    )
-    (property "Package" "None" (at 43.18 99.06 0)
-      (effects (font (size 1.27 1.27)) (justify bottom) hide)
-    )
-    (property "Check_prices" "https://www.snapeda.com/parts/BOB-12009/SparkFun+Electronics/view-part/?ref=eda" (at 43.18 99.06 0)
-      (effects (font (size 1.27 1.27)) (justify bottom) hide)
-    )
-    (property "STANDARD" "Manufacturer Recommendations" (at 43.18 99.06 0)
-      (effects (font (size 1.27 1.27)) (justify bottom) hide)
-    )
-    (property "PARTREV" "01" (at 43.18 99.06 0)
-      (effects (font (size 1.27 1.27)) (justify bottom) hide)
-    )
-    (property "SnapEDA_Link" "https://www.snapeda.com/parts/BOB-12009/SparkFun+Electronics/view-part/?ref=snap" (at 43.18 99.06 0)
-      (effects (font (size 1.27 1.27)) (justify bottom) hide)
-    )
-    (property "MP" "BOB-12009" (at 43.18 99.06 0)
-      (effects (font (size 1.27 1.27)) (justify bottom) hide)
-    )
-    (property "Purchase-URL" "https://pricing.snapeda.com/search?q=BOB-12009&ref=eda" (at 43.18 99.06 0)
-      (effects (font (size 1.27 1.27)) (justify bottom) hide)
-    )
-    (property "Description" "\nBSS138 Logic-Level Translator Interface Evaluation Board\n" (at 43.18 99.06 0)
-      (effects (font (size 1.27 1.27)) (justify bottom) hide)
-    )
-    (property "MANUFACTURER" "SparkFun Electronics" (at 43.18 99.06 0)
-      (effects (font (size 1.27 1.27)) (justify bottom) hide)
-    )
-    (pin "GND_1")
-    (pin "GND_2")
-    (pin "HV")
-    (pin "HV1")
-    (pin "HV2")
-    (pin "HV3")
-    (pin "HV4")
-    (pin "LV")
-    (pin "LV1")
-    (pin "LV2")
-    (pin "LV3")
-    (pin "LV4")
-    (instances
-      (project "INDY THE TREASURE HUNTER"
-        (path "/b3b90d4c-73f4-4a78-9e6e-dd19a1913646"
-          (reference "U?") (unit 1)
-        )
-      )
-    )
-  )
-  (symbol (lib_id "ARDUINO UNO:ABX00027") (at 92.71 77.47 0) (unit 1)
-    (in_bom yes) (on_board yes) (dnp no) (fields_autoplaced)
-    (property "Reference" "U?" (at 92.71 48.26 0)
-      (effects (font (size 1.27 1.27)))
-    )
-    (property "Value" "ARDUINO UNO" (at 92.71 50.8 0)
-      (effects (font (size 1.27 1.27)))
-    )
-    (property "Footprint" "MODULE_ABX00027" (at 91.44 124.46 0)
-      (effects (font (size 1.27 1.27)) (justify bottom) hide)
-    )
-    (property "Datasheet" "" (at 92.71 77.47 0)
-      (effects (font (size 1.27 1.27)) hide)
-    )
-    (property "MF" "Arduino" (at 91.44 132.08 0)
-      (effects (font (size 1.27 1.27)) (justify bottom) hide)
-    )
-    (property "DESCRIPTION" "ATSAMD21G18A Arduino Nano 33 IoT SAM D ARM® Cortex®-M0+ MCU 32-Bit Embedded Evaluation Board" (at 92.71 110.49 0)
-      (effects (font (size 1.27 1.27)) (justify bottom) hide)
-    )
-    (property "PACKAGE" "None" (at 91.44 133.35 0)
-      (effects (font (size 1.27 1.27)) (justify bottom) hide)
-    )
-    (property "PRICE" "None" (at 92.71 134.62 0)
-      (effects (font (size 1.27 1.27)) (justify bottom) hide)
-    )
-    (property "Package" "None" (at 82.55 127 0)
-      (effects (font (size 1.27 1.27)) (justify bottom) hide)
-    )
-    (property "Check_prices" "" (at 92.71 77.47 0)
-      (effects (font (size 1.27 1.27)) (justify bottom) hide)
-    )
-    (property "Price" "None" (at 82.55 127 0)
-      (effects (font (size 1.27 1.27)) (justify bottom) hide)
-    )
-    (property "SnapEDA_Link" "https://www.snapeda.com/parts/Arduino%20Nano%2033%20IoT/Arduino/view-part/?ref=snap" (at 95.25 118.11 0)
-      (effects (font (size 1.27 1.27)) (justify bottom) hide)
-    )
-    (property "MP" "Arduino Nano 33 IoT" (at 91.44 129.54 0)
-      (effects (font (size 1.27 1.27)) (justify bottom) hide)
-    )
-    (property "DIGIKEY-PURCHASE-URL" "https://snapeda.com/shop?store=DigiKey&id=3949339" (at 95.25 114.3 0)
-      (effects (font (size 1.27 1.27)) (justify bottom) hide)
-    )
-    (property "Availability" "Not in stock" (at 107.95 128.27 0)
-      (effects (font (size 1.27 1.27)) (justify bottom) hide)
-    )
-    (property "AVAILABILITY" "Unavailable" (at 82.55 127 0)
-      (effects (font (size 1.27 1.27)) (justify bottom) hide)
-    )
-    (property "Description" "\nAn IoT connected IMU sensor in the Nano form factor.\n" (at 88.9 121.92 0)
-      (effects (font (size 1.27 1.27)) (justify bottom) hide)
-    )
-    (pin "1")
-    (pin "10")
-    (pin "11")
-    (pin "12")
-    (pin "13")
-    (pin "14")
-    (pin "15")
-    (pin "16")
-    (pin "17")
-    (pin "18")
-    (pin "19")
-    (pin "2")
-    (pin "20")
-    (pin "21")
-    (pin "22")
-    (pin "23")
-    (pin "24")
-    (pin "25")
-    (pin "26")
-    (pin "27")
-    (pin "28")
-    (pin "29")
-    (pin "3")
-    (pin "30")
-    (pin "4")
-    (pin "5")
-    (pin "6")
-    (pin "7")
-    (pin "8")
-    (pin "9")
-    (instances
-      (project "INDY THE TREASURE HUNTER"
-        (path "/b3b90d4c-73f4-4a78-9e6e-dd19a1913646"
-          (reference "U?") (unit 1)
-        )
-      )
-    )
-  )
-  (symbol (lib_id "BOB-12009:BOB-12009") (at 43.18 67.31 0) (unit 1)
-    (in_bom yes) (on_board yes) (dnp no) (fields_autoplaced)
-    (property "Reference" "U?" (at 43.18 53.34 0)
-      (effects (font (size 1.27 1.27)))
-    )
-    (property "Value" "BOB-12009" (at 43.18 55.88 0)
-      (effects (font (size 1.27 1.27)))
-    )
-    (property "Footprint" "CONV_BOB-12009" (at 43.18 67.31 0)
-      (effects (font (size 1.27 1.27)) (justify bottom) hide)
-    )
-    (property "Datasheet" "" (at 43.18 67.31 0)
-      (effects (font (size 1.27 1.27)) hide)
-    )
-    (property "DigiKey_Part_Number" "1568-1209-ND" (at 43.18 67.31 0)
-      (effects (font (size 1.27 1.27)) (justify bottom) hide)
-    )
-    (property "MF" "SparkFun" (at 43.18 67.31 0)
-      (effects (font (size 1.27 1.27)) (justify bottom) hide)
-    )
-    (property "MAXIMUM_PACKAGE_HEIGHT" "N/A" (at 43.18 67.31 0)
-      (effects (font (size 1.27 1.27)) (justify bottom) hide)
-    )
-    (property "Package" "None" (at 43.18 67.31 0)
-      (effects (font (size 1.27 1.27)) (justify bottom) hide)
-    )
-    (property "Check_prices" "https://www.snapeda.com/parts/BOB-12009/SparkFun+Electronics/view-part/?ref=eda" (at 43.18 67.31 0)
-      (effects (font (size 1.27 1.27)) (justify bottom) hide)
-    )
-    (property "STANDARD" "Manufacturer Recommendations" (at 43.18 67.31 0)
-      (effects (font (size 1.27 1.27)) (justify bottom) hide)
-    )
-    (property "PARTREV" "01" (at 43.18 67.31 0)
-      (effects (font (size 1.27 1.27)) (justify bottom) hide)
-    )
-    (property "SnapEDA_Link" "https://www.snapeda.com/parts/BOB-12009/SparkFun+Electronics/view-part/?ref=snap" (at 43.18 67.31 0)
-      (effects (font (size 1.27 1.27)) (justify bottom) hide)
-    )
-    (property "MP" "BOB-12009" (at 43.18 67.31 0)
-      (effects (font (size 1.27 1.27)) (justify bottom) hide)
-    )
-    (property "Purchase-URL" "https://pricing.snapeda.com/search?q=BOB-12009&ref=eda" (at 43.18 67.31 0)
-      (effects (font (size 1.27 1.27)) (justify bottom) hide)
-    )
-    (property "Description" "\nBSS138 Logic-Level Translator Interface Evaluation Board\n" (at 43.18 67.31 0)
-      (effects (font (size 1.27 1.27)) (justify bottom) hide)
-    )
-    (property "MANUFACTURER" "SparkFun Electronics" (at 43.18 67.31 0)
-      (effects (font (size 1.27 1.27)) (justify bottom) hide)
-    )
-    (pin "GND_1")
-    (pin "GND_2")
-    (pin "HV")
-    (pin "HV1")
-    (pin "HV2")
-    (pin "HV3")
-    (pin "HV4")
-    (pin "LV")
-    (pin "LV1")
-    (pin "LV2")
-    (pin "LV3")
-    (pin "LV4")
-    (instances
-      (project "INDY THE TREASURE HUNTER"
-        (path "/b3b90d4c-73f4-4a78-9e6e-dd19a1913646"
-          (reference "U?") (unit 1)
-        )
-      )
-    )
-  )
   (sheet (at 173.99 48.26) (size 57.15 36.83) (fields_autoplaced)
     (stroke (width 0.1524) (type solid))
@@
       )
     )
+  )
+  (sheet (at 21.59 44.45) (size 101.6 78.74) (fields_autoplaced)
+    (stroke (width 0.1524) (type solid))
+    (fill (color 0 0 0 0.0000))
+    (property "Sheetname" "MICROCONTROLLER" (at 21.59 43.7384 0)
+      (effects (font (size 1.27 1.27)) (justify left bottom))
+    )
+    (property "Sheetfile" "MICROCONTROLLER.kicad_sch" (at 21.59 123.7746 0)
+      (effects (font (size 1.27 1.27)) (justify left top))
+    )
+    (instances
+      (project "INDY THE TREASURE HUNTER"
+        (path "/b3b90d4c-73f4-4a78-9e6e-dd19a1913646" (page "3"))
+      )
+    )

Commit message: .
Other:
- added sheet MOTOR (MOTOR.kicad_sch)
- added sheet POWER (POWER.kicad_sch)
Changed lines of the file:
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@@
 (kicad_sch (version 20230121) (generator eeschema)
   (paper "A4")
-  (sheet (at 173.99 48.26) (size 57.15 36.83) (fields_autoplaced)
+  (hierarchical_label "3V3" (shape input) (at 194.31 104.14 0) (fields_autoplaced)
+    (effects (font (size 1.27 1.27)) (justify left))
+  )
+  (sheet (at 40.64 97.79) (size 77.47 39.37) (fields_autoplaced)
     (stroke (width 0.1524) (type solid))
     (fill (color 0 0 0 0.0000))
-    (property "Sheetname" "SENSING" (at 173.99 47.5484 0)
+    (property "Sheetname" "MOTOR" (at 40.64 97.0784 0)
       (effects (font (size 1.27 1.27)) (justify left bottom))
     )
-    (property "Sheetfile" "SENSING.kicad_sch" (at 173.99 85.6746 0)
+    (property "Sheetfile" "MOTOR.kicad_sch" (at 40.64 137.7446 0)
+      (effects (font (size 1.27 1.27)) (justify left top))
+    )
+    (instances
+      (project "INDY THE TREASURE HUNTER"
+        (path "/b3b90d4c-73f4-4a78-9e6e-dd19a1913646" (page "4"))
+      )
+    )
+  )
+  (sheet (at 132.08 41.91) (size 57.15 36.83) (fields_autoplaced)
+    (stroke (width 0.1524) (type solid))
+    (fill (color 0 0 0 0.0000))
+    (property "Sheetname" "SENSING" (at 132.08 41.1984 0)
+      (effects (font (size 1.27 1.27)) (justify left bottom))
+    )
+    (property "Sheetfile" "SENSING.kicad_sch" (at 132.08 79.3246 0)
       (effects (font (size 1.27 1.27)) (justify left top))
     )
@@
     )
   )
-  (sheet (at 21.59 44.45) (size 101.6 78.74) (fields_autoplaced)
+  (sheet (at 38.1 40.64) (size 77.47 41.91) (fields_autoplaced)
     (stroke (width 0.1524) (type solid))
     (fill (color 0 0 0 0.0000))
-    (property "Sheetname" "MICROCONTROLLER" (at 21.59 43.7384 0)
+    (property "Sheetname" "MICROCONTROLLER" (at 38.1 39.9284 0)
       (effects (font (size 1.27 1.27)) (justify left bottom))
     )
-    (property "Sheetfile" "MICROCONTROLLER.kicad_sch" (at 21.59 123.7746 0)
+    (property "Sheetfile" "MICROCONTROLLER.kicad_sch" (at 38.1 83.1346 0)
       (effects (font (size 1.27 1.27)) (justify left top))
     )
@@
       )
     )
+  )
+  (sheet (at 132.08 97.79) (size 62.23 39.37) (fields_autoplaced)
+    (stroke (width 0.1524) (type solid))
+    (fill (color 0 0 0 0.0000))
+    (property "Sheetname" "POWER" (at 132.08 97.0784 0)
+      (effects (font (size 1.27 1.27)) (justify left bottom))
+    )
+    (property "Sheetfile" "POWER.kicad_sch" (at 132.08 137.7446 0)
+      (effects (font (size 1.27 1.27)) (justify left top))
+    )
+    (instances
+      (project "INDY THE TREASURE HUNTER"
+        (path "/b3b90d4c-73f4-4a78-9e6e-dd19a1913646" (page "5"))
+      )
+    )

Commit message: .
Changed lines of the file:
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@@
 (kicad_sch (version 20230121) (generator eeschema)
   (paper "A4")
+  (wire (pts (xy 189.23 67.31) (xy 194.31 104.14))
+    (stroke (width 0) (type default))
+  )
+  (hierarchical_label "3V3" (shape input) (at 189.23 67.31 0) (fields_autoplaced)
+    (effects (font (size 1.27 1.27)) (justify left))
+  )
   (hierarchical_label "3V3" (shape input) (at 194.31 104.14 0) (fields_autoplaced)
     (effects (font (size 1.27 1.27)) (justify left))
@@
     )
   )
-  (sheet (at 132.08 97.79) (size 62.23 39.37) (fields_autoplaced)
+  (sheet (at 132.08 102.87) (size 62.23 39.37) (fields_autoplaced)
     (stroke (width 0.1524) (type solid))
     (fill (color 0 0 0 0.0000))
-    (property "Sheetname" "POWER" (at 132.08 97.0784 0)
+    (property "Sheetname" "POWER" (at 132.08 102.1584 0)
       (effects (font (size 1.27 1.27)) (justify left bottom))
     )
-    (property "Sheetfile" "POWER.kicad_sch" (at 132.08 137.7446 0)
+    (property "Sheetfile" "POWER.kicad_sch" (at 132.08 142.8246 0)
       (effects (font (size 1.27 1.27)) (justify left top))
     )
