File: INDY THE TREASURE HUNTER/INDY THE TREASURE HUNTER.kicad_sch (KiCad schematic)
At the start: 0 parts

Commit message: 17:32
Changed lines of the file:
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@@
 (kicad_sch (version 20230121) (generator eeschema)
   (paper "A4")
+  (wire (pts (xy 193.04 109.22) (xy 208.28 109.22))
+    (stroke (width 0) (type default))
+  )
+  (wire (pts (xy 208.28 109.22) (xy 208.28 44.45))
+    (stroke (width 0) (type default))
+  )
+  (wire (pts (xy 193.04 44.45) (xy 208.28 44.45))
+    (stroke (width 0) (type default))
+  )
+  (hierarchical_label "5V" (shape input) (at 193.04 44.45 180) (fields_autoplaced)
+    (effects (font (size 1.27 1.27)) (justify right))
+  )
   (hierarchical_label "3V3OUT" (shape output) (at 115.57 44.45 180) (fields_autoplaced)
     (effects (font (size 1.27 1.27)) (justify right))
@@
     (effects (font (size 1.27 1.27)) (justify right))
   )
+  (hierarchical_label "5V" (shape output) (at 193.04 109.22 180) (fields_autoplaced)
+    (effects (font (size 1.27 1.27)) (justify right))
+  )
