File: INDY THE TREASURE HUNTER/MICROCONTROLLER.kicad_sch (KiCad schematic)
At the start: 3 parts

Commit message: .
Connections:
- net GND: now reaches U?.14 (GND), U?.19 (GND)
- net GND: now also U?.GND_1 (GND), U?.GND_1 (GND), U?.GND_2 (GND), U?.GND_2 (GND)
Other:
- moved on the sheet: U?

Commit message: .
Other:
- moved on the sheet: U?
