File: INDY THE TREASURE HUNTER/MICROCONTROLLER.kicad_sch (KiCad schematic)
At the start: 3 parts

Commit message: 17:32
Other:
- note added: "DO NOT CONNECT A 5V SIGNAL TO THIS BOARD OR IT DIES"
- moved on the sheet: U?
Changed lines of the file:
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@@
     (stroke (width 0) (type default))
   )
-  (wire (pts (xy 196.85 83.82) (xy 196.85 111.76))
+  (wire (pts (xy 196.85 80.01) (xy 196.85 111.76))
     (stroke (width 0) (type default))
   )
@@
     (stroke (width 0) (type default))
   )
-  (wire (pts (xy 196.85 83.82) (xy 195.58 83.82))
+  (wire (pts (xy 196.85 80.01) (xy 194.31 80.01))
     (stroke (width 0) (type default))
   )
@@
     (stroke (width 0) (type default))
   )
-  (symbol (lib_id "ARDUINO UNO:ABX00027") (at 177.8 60.96 0) (unit 1)
-    (in_bom yes) (on_board yes) (dnp no) (fields_autoplaced)
-    (property "Reference" "U?" (at 177.8 31.75 0)
-      (effects (font (size 1.27 1.27)))
-    )
-    (property "Value" "ARDUINO UNO" (at 177.8 34.29 0)
-      (effects (font (size 1.27 1.27)))
-    )
-    (property "Footprint" "MODULE_ABX00027" (at 176.53 107.95 0)
-      (effects (font (size 1.27 1.27)) (justify bottom) hide)
-    )
-    (property "Datasheet" "" (at 177.8 60.96 0)
-      (effects (font (size 1.27 1.27)) hide)
-    )
-    (property "MF" "Arduino" (at 176.53 115.57 0)
-      (effects (font (size 1.27 1.27)) (justify bottom) hide)
-    )
-    (property "DESCRIPTION" "ATSAMD21G18A Arduino Nano 33 IoT SAM D ARM® Cortex®-M0+ MCU 32-Bit Embedded Evaluation Board" (at 177.8 93.98 0)
-      (effects (font (size 1.27 1.27)) (justify bottom) hide)
-    )
-    (property "PACKAGE" "None" (at 176.53 116.84 0)
-      (effects (font (size 1.27 1.27)) (justify bottom) hide)
-    )
-    (property "PRICE" "None" (at 177.8 118.11 0)
-      (effects (font (size 1.27 1.27)) (justify bottom) hide)
-    )
-    (property "Package" "None" (at 167.64 110.49 0)
-      (effects (font (size 1.27 1.27)) (justify bottom) hide)
-    )
-    (property "Check_prices" "" (at 177.8 60.96 0)
-      (effects (font (size 1.27 1.27)) (justify bottom) hide)
-    )
-    (property "Price" "None" (at 167.64 110.49 0)
-      (effects (font (size 1.27 1.27)) (justify bottom) hide)
-    )
-    (property "SnapEDA_Link" "https://www.snapeda.com/parts/Arduino%20Nano%2033%20IoT/Arduino/view-part/?ref=snap" (at 180.34 101.6 0)
-      (effects (font (size 1.27 1.27)) (justify bottom) hide)
-    )
-    (property "MP" "Arduino Nano 33 IoT" (at 176.53 113.03 0)
-      (effects (font (size 1.27 1.27)) (justify bottom) hide)
-    )
-    (property "DIGIKEY-PURCHASE-URL" "https://snapeda.com/shop?store=DigiKey&id=3949339" (at 180.34 97.79 0)
-      (effects (font (size 1.27 1.27)) (justify bottom) hide)
-    )
-    (property "Availability" "Not in stock" (at 193.04 111.76 0)
-      (effects (font (size 1.27 1.27)) (justify bottom) hide)
-    )
-    (property "AVAILABILITY" "Unavailable" (at 167.64 110.49 0)
-      (effects (font (size 1.27 1.27)) (justify bottom) hide)
-    )
-    (property "Description" "\nAn IoT connected IMU sensor in the Nano form factor.\n" (at 173.99 105.41 0)
+  (text "DO NOT CONNECT A 5V SIGNAL TO THIS BOARD OR IT DIES"
+    (at 151.13 25.4 0)
+    (effects (font (size 1.27 1.27)) (justify left bottom))
+  )
+  (symbol (lib_id "ARDUINO UNO:ABX00027") (at 176.53 57.15 0) (unit 1)
+    (in_bom yes) (on_board yes) (dnp no) (fields_autoplaced)
+    (property "Reference" "U?" (at 176.53 27.94 0)
+      (effects (font (size 1.27 1.27)))
+    )
+    (property "Value" "ARDUINO UNO" (at 176.53 30.48 0)
+      (effects (font (size 1.27 1.27)))
+    )
+    (property "Footprint" "MODULE_ABX00027" (at 175.26 104.14 0)
+      (effects (font (size 1.27 1.27)) (justify bottom) hide)
+    )
+    (property "Datasheet" "" (at 176.53 57.15 0)
+      (effects (font (size 1.27 1.27)) hide)
+    )
+    (property "MF" "Arduino" (at 175.26 111.76 0)
+      (effects (font (size 1.27 1.27)) (justify bottom) hide)
+    )
+    (property "DESCRIPTION" "ATSAMD21G18A Arduino Nano 33 IoT SAM D ARM® Cortex®-M0+ MCU 32-Bit Embedded Evaluation Board" (at 176.53 90.17 0)
+      (effects (font (size 1.27 1.27)) (justify bottom) hide)
+    )
+    (property "PACKAGE" "None" (at 175.26 113.03 0)
+      (effects (font (size 1.27 1.27)) (justify bottom) hide)
+    )
+    (property "PRICE" "None" (at 176.53 114.3 0)
+      (effects (font (size 1.27 1.27)) (justify bottom) hide)
+    )
+    (property "Package" "None" (at 166.37 106.68 0)
+      (effects (font (size 1.27 1.27)) (justify bottom) hide)
+    )
+    (property "Check_prices" "" (at 176.53 57.15 0)
+      (effects (font (size 1.27 1.27)) (justify bottom) hide)
+    )
+    (property "Price" "None" (at 166.37 106.68 0)
+      (effects (font (size 1.27 1.27)) (justify bottom) hide)
+    )
+    (property "SnapEDA_Link" "https://www.snapeda.com/parts/Arduino%20Nano%2033%20IoT/Arduino/view-part/?ref=snap" (at 179.07 97.79 0)
+      (effects (font (size 1.27 1.27)) (justify bottom) hide)
+    )
+    (property "MP" "Arduino Nano 33 IoT" (at 175.26 109.22 0)
+      (effects (font (size 1.27 1.27)) (justify bottom) hide)
+    )
+    (property "DIGIKEY-PURCHASE-URL" "https://snapeda.com/shop?store=DigiKey&id=3949339" (at 179.07 93.98 0)
+      (effects (font (size 1.27 1.27)) (justify bottom) hide)
+    )
+    (property "Availability" "Not in stock" (at 191.77 107.95 0)
+      (effects (font (size 1.27 1.27)) (justify bottom) hide)
+    )
+    (property "AVAILABILITY" "Unavailable" (at 166.37 106.68 0)
+      (effects (font (size 1.27 1.27)) (justify bottom) hide)
+    )
+    (property "Description" "\nAn IoT connected IMU sensor in the Nano form factor.\n" (at 172.72 101.6 0)
       (effects (font (size 1.27 1.27)) (justify bottom) hide)
     )
@@
         )
         (path "/b3b90d4c-73f4-4a78-9e6e-dd19a1913646/a6eb79ec-4315-4230-a936-5681391aafb7"
-          (reference "U?") (unit 1)
+          (reference "U4") (unit 1)
         )
       )
@@
         )
         (path "/b3b90d4c-73f4-4a78-9e6e-dd19a1913646/a6eb79ec-4315-4230-a936-5681391aafb7"
-          (reference "U?") (unit 1)
+          (reference "U3") (unit 1)
         )
       )
@@
         )
         (path "/b3b90d4c-73f4-4a78-9e6e-dd19a1913646/a6eb79ec-4315-4230-a936-5681391aafb7"
-          (reference "U?") (unit 1)
-        )
-      )
+          (reference "U2") (unit 1)
+        )
+      )
