File: INDY THE TREASURE HUNTER/MICROCONTROLLER.kicad_sch (KiCad schematic)
At the start: 3 parts

Commit message: Wired up Ultrasonic sensor
I think the USonic sensor is wired up completely. Not that bad actually.
Connections:
- net D7: now reaches U?.25 (D7)
- net D8: now reaches U?.26 (D8)
Other:
- note added: "The datasheet specifies that some pins here have more functions than just GPIO. Lets try fill up the ONLY GPIO pins first, before colonizing other pins"
Changed lines of the file:
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@@
+    (stroke (width 0) (type default))
+  )
+  (wire (pts (xy 194.31 57.15) (xy 198.12 57.15))
     (stroke (width 0) (type default))
   )
   (wire (pts (xy 196.85 80.01) (xy 196.85 111.76))
+    (stroke (width 0) (type default))
+  )
+  (wire (pts (xy 194.31 59.69) (xy 198.12 59.69))
     (stroke (width 0) (type default))
   )
@@
     (stroke (width 0) (type default))
   )
+  (text "The datasheet specifies that some pins here have more\nfunctions than just GPIO. Lets try fill up the ONLY GPIO\npins first, before colonizing other pins"
+    (at 210.82 39.37 0)
+    (effects (font (size 1.27 1.27)) (justify left bottom))
+  )
   (text "DO NOT CONNECT A 5V SIGNAL TO THIS BOARD OR IT DIES"
     (at 151.13 25.4 0)
     (effects (font (size 1.27 1.27)) (justify left bottom))
   )
+  (hierarchical_label "D8" (shape input) (at 198.12 59.69 0) (fields_autoplaced)
+    (effects (font (size 1.27 1.27)) (justify left))
+  )
+  (hierarchical_label "D7" (shape output) (at 198.12 57.15 0) (fields_autoplaced)
+    (effects (font (size 1.27 1.27)) (justify left))
+  )
   (hierarchical_label "3V3IN" (shape input) (at 198.12 34.29 0) (fields_autoplaced)

Commit message: Line sensor data lines configured
Im pretty sure the line sensors operate fine on 3v3, so no need to shift their logic levels or anything
Connections:
- net D2: now reaches U?.20 (D2)
- net D3: now reaches U?.21 (D3/PWM)
- net D4: now reaches U?.22 (D4)
- net D5: now reaches U?.23 (D5/PWM)
Changed lines of the file:
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@@
+    (stroke (width 0) (type default))
+  )
+  (wire (pts (xy 194.31 46.99) (xy 198.12 46.99))
     (stroke (width 0) (type default))
   )
@@
   )
   (wire (pts (xy 196.85 111.76) (xy 160.02 111.76))
+    (stroke (width 0) (type default))
+  )
+  (wire (pts (xy 194.31 52.07) (xy 198.12 52.07))
+    (stroke (width 0) (type default))
+  )
+  (wire (pts (xy 194.31 44.45) (xy 198.12 44.45))
     (stroke (width 0) (type default))
   )
@@
   )
   (wire (pts (xy 160.02 111.76) (xy 160.02 116.84))
+    (stroke (width 0) (type default))
+  )
+  (wire (pts (xy 194.31 49.53) (xy 198.12 49.53))
     (stroke (width 0) (type default))
   )
@@
     (effects (font (size 1.27 1.27)) (justify left))
   )
+  (hierarchical_label "D3" (shape input) (at 198.12 46.99 0) (fields_autoplaced)
+    (effects (font (size 1.27 1.27)) (justify left))
+  )
   (hierarchical_label "D7" (shape output) (at 198.12 57.15 0) (fields_autoplaced)
     (effects (font (size 1.27 1.27)) (justify left))
   )
+  (hierarchical_label "D2" (shape input) (at 198.12 44.45 0) (fields_autoplaced)
+    (effects (font (size 1.27 1.27)) (justify left))
+  )
+  (hierarchical_label "D4" (shape input) (at 198.12 49.53 0) (fields_autoplaced)
+    (effects (font (size 1.27 1.27)) (justify left))
+  )
+  (hierarchical_label "D5" (shape input) (at 198.12 52.07 0) (fields_autoplaced)
+    (effects (font (size 1.27 1.27)) (justify left))
+  )

Commit message: I think thats that?
There are a few things that remain unclear. For milestone 1's handin, it should be ok, just some cleanup in the morning might be necessary and group discussion on how to do things
Other:
- note added: "No idea what these are, I might be missing something? OH literally as Im typing this I see theyre the logic level shifters Um... we can decide to use headers later this isnt a final design"
Changed lines of the file:
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@@
     (stroke (width 0) (type default))
+  )
+  (rectangle (start 83.185 27.94) (end 142.875 124.46)
+    (stroke (width 0) (type default))
+    (fill (type none))
   )
   (text "The datasheet specifies that some pins here have more\nfunctions than just GPIO. Lets try fill up the ONLY GPIO\npins first, before colonizing other pins"
@@
     (effects (font (size 1.27 1.27)) (justify left bottom))
   )
+  (text "No idea what these are, I might be missing something? OH literally \nas Im typing this I see theyre the logic level shifters\n\nUm... we can decide to use headers later this isnt a final design"
+    (at 78.74 26.035 0)
+    (effects (font (size 1.27 1.27)) (justify left bottom))
+  )

Commit message: Neatened up schematic for milestone 1 handin
Parts:
- removed U? (x2): BOB-12009, CONV_BOB-12009, symbol BOB-12009:BOB-12009
Other:
- note removed: "No idea what these are, I might be missing something? OH literally as Im typing this I see theyre the logic level shifters Um... we can decide to use headers later this isnt a final design"
Changed lines of the file:
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@@
 (kicad_sch (version 20230121) (generator eeschema)
   (paper "A4")
-  (junction (at 148.59 111.76) (diameter 0) (color 0 0 0 0)
-  )
-  (junction (at 160.02 111.76) (diameter 0) (color 0 0 0 0)
-  )
   (wire (pts (xy 194.31 39.37) (xy 198.12 39.37))
     (stroke (width 0) (type default))
   )
-  (wire (pts (xy 148.59 54.61) (xy 148.59 111.76))
-    (stroke (width 0) (type default))
-  )
   (wire (pts (xy 194.31 57.15) (xy 198.12 57.15))
-    (stroke (width 0) (type default))
-  )
-  (wire (pts (xy 196.85 80.01) (xy 196.85 111.76))
     (stroke (width 0) (type default))
   )
@@
     (stroke (width 0) (type default))
   )
-  (wire (pts (xy 148.59 111.76) (xy 160.02 111.76))
-    (stroke (width 0) (type default))
-  )
-  (wire (pts (xy 196.85 111.76) (xy 160.02 111.76))
-    (stroke (width 0) (type default))
-  )
   (wire (pts (xy 194.31 52.07) (xy 198.12 52.07))
     (stroke (width 0) (type default))
@@
     (stroke (width 0) (type default))
   )
-  (wire (pts (xy 148.59 54.61) (xy 130.81 54.61))
-    (stroke (width 0) (type default))
-  )
-  (wire (pts (xy 196.85 80.01) (xy 194.31 80.01))
-    (stroke (width 0) (type default))
-  )
-  (wire (pts (xy 160.02 111.76) (xy 160.02 116.84))
+  (wire (pts (xy 194.31 80.01) (xy 200.66 80.01))
     (stroke (width 0) (type default))
   )
@@
     (stroke (width 0) (type default))
   )
+  (wire (pts (xy 200.66 80.01) (xy 200.66 83.185))
+    (stroke (width 0) (type default))
+  )
   (wire (pts (xy 194.31 34.29) (xy 198.12 34.29))
     (stroke (width 0) (type default))
   )
-  (wire (pts (xy 130.81 111.76) (xy 148.59 111.76))
-    (stroke (width 0) (type default))
-  )
-  (rectangle (start 83.185 27.94) (end 142.875 124.46)
-    (stroke (width 0) (type default))
-    (fill (type none))
-  )
   (text "The datasheet specifies that some pins here have more\nfunctions than just GPIO. Lets try fill up the ONLY GPIO\npins first, before colonizing other pins"
     (at 210.82 39.37 0)
-    (effects (font (size 1.27 1.27)) (justify left bottom))
-  )
-  (text "No idea what these are, I might be missing something? OH literally \nas Im typing this I see theyre the logic level shifters\n\nUm... we can decide to use headers later this isnt a final design"
-    (at 78.74 26.035 0)
     (effects (font (size 1.27 1.27)) (justify left bottom))
   )
@@
     )
   )
-  (symbol (lib_name "BOB-12009_1") (lib_id "BOB-12009:BOB-12009") (at 113.03 101.6 0) (unit 1)
+  (symbol (lib_id "power:GND") (at 200.66 83.185 0) (unit 1)
     (in_bom yes) (on_board yes) (dnp no) (fields_autoplaced)
-    (property "Reference" "U?" (at 113.03 87.63 0)
+    (property "Reference" "#PWR01" (at 200.66 89.535 0)
+      (effects (font (size 1.27 1.27)) hide)
+    )
+    (property "Value" "GND" (at 200.66 88.265 0)
       (effects (font (size 1.27 1.27)))
     )
-    (property "Value" "BOB-12009" (at 113.03 90.17 0)
-      (effects (font (size 1.27 1.27)))
-    )
-    (property "Footprint" "CONV_BOB-12009" (at 113.03 101.6 0)
-      (effects (font (size 1.27 1.27)) (justify bottom) hide)
-    )
-    (property "Datasheet" "" (at 113.03 101.6 0)
+    (property "Footprint" "" (at 200.66 83.185 0)
       (effects (font (size 1.27 1.27)) hide)
     )
-    (property "DigiKey_Part_Number" "1568-1209-ND" (at 113.03 101.6 0)
-      (effects (font (size 1.27 1.27)) (justify bottom) hide)
-    )
-    (property "MF" "SparkFun" (at 113.03 101.6 0)
-      (effects (font (size 1.27 1.27)) (justify bottom) hide)
-    )
-    (property "MAXIMUM_PACKAGE_HEIGHT" "N/A" (at 113.03 101.6 0)
-      (effects (font (size 1.27 1.27)) (justify bottom) hide)
-    )
-    (property "Package" "None" (at 113.03 101.6 0)
-      (effects (font (size 1.27 1.27)) (justify bottom) hide)
-    )
-    (property "Check_prices" "https://www.snapeda.com/parts/BOB-12009/SparkFun+Electronics/view-part/?ref=eda" (at 113.03 101.6 0)
-      (effects (font (size 1.27 1.27)) (justify bottom) hide)
-    )
-    (property "STANDARD" "Manufacturer Recommendations" (at 113.03 101.6 0)
-      (effects (font (size 1.27 1.27)) (justify bottom) hide)
-    )
-    (property "PARTREV" "01" (at 113.03 101.6 0)
-      (effects (font (size 1.27 1.27)) (justify bottom) hide)
-    )
-    (property "SnapEDA_Link" "https://www.snapeda.com/parts/BOB-12009/SparkFun+Electronics/view-part/?ref=snap" (at 113.03 101.6 0)
-      (effects (font (size 1.27 1.27)) (justify bottom) hide)
-    )
-    (property "MP" "BOB-12009" (at 113.03 101.6 0)
-      (effects (font (size 1.27 1.27)) (justify bottom) hide)
-    )
-    (property "Purchase-URL" "https://pricing.snapeda.com/search?q=BOB-12009&ref=eda" (at 113.03 101.6 0)
-      (effects (font (size 1.27 1.27)) (justify bottom) hide)
-    )
-    (property "Description" "\nBSS138 Logic-Level Translator Interface Evaluation Board\n" (at 113.03 101.6 0)
-      (effects (font (size 1.27 1.27)) (justify bottom) hide)
-    )
-    (property "MANUFACTURER" "SparkFun Electronics" (at 113.03 101.6 0)
-      (effects (font (size 1.27 1.27)) (justify bottom) hide)
-    )
-    (pin "GND_1")
-    (pin "GND_2")
-    (pin "HV")
-    (pin "HV1")
-    (pin "HV2")
-    (pin "HV3")
-    (pin "HV4")
-    (pin "LV")
-    (pin "LV1")
-    (pin "LV2")
-    (pin "LV3")
-    (pin "LV4")
-    (instances
-      (project "INDY THE TREASURE HUNTER"
-        (path "/b3b90d4c-73f4-4a78-9e6e-dd19a1913646"
-          (reference "U?") (unit 1)
-        )
-        (path "/b3b90d4c-73f4-4a78-9e6e-dd19a1913646/a6eb79ec-4315-4230-a936-5681391aafb7"
-          (reference "U3") (unit 1)
-        )
-      )
-    )
-  )
-  (symbol (lib_id "power:GND") (at 160.02 116.84 0) (unit 1)
-    (in_bom yes) (on_board yes) (dnp no) (fields_autoplaced)
-    (property "Reference" "#PWR01" (at 160.02 123.19 0)
-      (effects (font (size 1.27 1.27)) hide)
-    )
-    (property "Value" "GND" (at 160.02 121.92 0)
-      (effects (font (size 1.27 1.27)))
-    )
-    (property "Footprint" "" (at 160.02 116.84 0)
-      (effects (font (size 1.27 1.27)) hide)
-    )
-    (property "Datasheet" "" (at 160.02 116.84 0)
+    (property "Datasheet" "" (at 200.66 83.185 0)
       (effects (font (size 1.27 1.27)) hide)
     )
@@
         )
       )
-    )
-  )
-  (symbol (lib_id "BOB-12009:BOB-12009") (at 113.03 44.45 0) (unit 1)
-    (in_bom yes) (on_board yes) (dnp no) (fields_autoplaced)
-    (property "Reference" "U?" (at 113.03 30.48 0)
-      (effects (font (size 1.27 1.27)))
-    )
-    (property "Value" "BOB-12009" (at 113.03 33.02 0)
-      (effects (font (size 1.27 1.27)))
-    )
-    (property "Footprint" "CONV_BOB-12009" (at 113.03 44.45 0)
-      (effects (font (size 1.27 1.27)) (justify bottom) hide)
-    )
-    (property "Datasheet" "" (at 113.03 44.45 0)
-      (effects (font (size 1.27 1.27)) hide)
-    )
-    (property "DigiKey_Part_Number" "1568-1209-ND" (at 113.03 44.45 0)
-      (effects (font (size 1.27 1.27)) (justify bottom) hide)
-    )
-    (property "MF" "SparkFun" (at 113.03 44.45 0)
-      (effects (font (size 1.27 1.27)) (justify bottom) hide)
-    )
-    (property "MAXIMUM_PACKAGE_HEIGHT" "N/A" (at 113.03 44.45 0)
-      (effects (font (size 1.27 1.27)) (justify bottom) hide)
-    )
-    (property "Package" "None" (at 113.03 44.45 0)
-      (effects (font (size 1.27 1.27)) (justify bottom) hide)
-    )
-    (property "Check_prices" "https://www.snapeda.com/parts/BOB-12009/SparkFun+Electronics/view-part/?ref=eda" (at 113.03 44.45 0)
-      (effects (font (size 1.27 1.27)) (justify bottom) hide)
-    )
-    (property "STANDARD" "Manufacturer Recommendations" (at 113.03 44.45 0)
-      (effects (font (size 1.27 1.27)) (justify bottom) hide)
-    )
-    (property "PARTREV" "01" (at 113.03 44.45 0)
-      (effects (font (size 1.27 1.27)) (justify bottom) hide)
-    )
-    (property "SnapEDA_Link" "https://www.snapeda.com/parts/BOB-12009/SparkFun+Electronics/view-part/?ref=snap" (at 113.03 44.45 0)
-      (effects (font (size 1.27 1.27)) (justify bottom) hide)
-    )
-    (property "MP" "BOB-12009" (at 113.03 44.45 0)
-      (effects (font (size 1.27 1.27)) (justify bottom) hide)
-    )
-    (property "Purchase-URL" "https://pricing.snapeda.com/search?q=BOB-12009&ref=eda" (at 113.03 44.45 0)
-      (effects (font (size 1.27 1.27)) (justify bottom) hide)
-    )
-    (property "Description" "\nBSS138 Logic-Level Translator Interface Evaluation Board\n" (at 113.03 44.45 0)
-      (effects (font (size 1.27 1.27)) (justify bottom) hide)
-    )
-    (property "MANUFACTURER" "SparkFun Electronics" (at 113.03 44.45 0)
-      (effects (font (size 1.27 1.27)) (justify bottom) hide)
-    )
-    (pin "GND_1")
-    (pin "GND_2")
-    (pin "HV")
-    (pin "HV1")
-    (pin "HV2")
-    (pin "HV3")
-    (pin "HV4")
-    (pin "LV")
-    (pin "LV1")
-    (pin "LV2")
-    (pin "LV3")
-    (pin "LV4")
-    (instances
-      (project "INDY THE TREASURE HUNTER"
-        (path "/b3b90d4c-73f4-4a78-9e6e-dd19a1913646"
-          (reference "U?") (unit 1)
-        )
-        (path "/b3b90d4c-73f4-4a78-9e6e-dd19a1913646/a6eb79ec-4315-4230-a936-5681391aafb7"
-          (reference "U2") (unit 1)
-        )
-      )

Commit message: No 3V3 regulator
Connections:
- net 3V3IN renamed 5V
Changed lines of the file:
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@@
     (effects (font (size 1.27 1.27)) (justify left))
   )
-  (hierarchical_label "3V3IN" (shape input) (at 198.12 34.29 0) (fields_autoplaced)
+  (hierarchical_label "5V" (shape input) (at 198.12 34.29 0) (fields_autoplaced)
     (effects (font (size 1.27 1.27)) (justify left))
   )
