File: INDY THE TREASURE HUNTER/SENSING.kicad_sch (KiCad schematic)
At the start: 1 part

Commit message: .
Changed lines of the file:
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@@
 (kicad_sch (version 20230121) (generator eeschema)
   (paper "A4")
-  (rectangle (start 59.69 44.45) (end 105.41 82.55)
+  (rectangle (start 83.82 40.64) (end 129.54 78.74)
     (stroke (width 0) (type default))
     (fill (type none))
   )
-  (rectangle (start 57.15 114.3) (end 106.68 160.02)
+  (rectangle (start 81.28 102.87) (end 130.81 148.59)
     (stroke (width 0) (type default))
     (fill (type none))
@@
     (fill (type none))
   )
-  (text "LINE SENSORS\n" (at 74.93 43.18 0)
+  (text "LINE SENSORS\n" (at 99.06 39.37 0)
     (effects (font (size 1.27 1.27)) (justify left bottom))
   )
@@
     (effects (font (size 1.27 1.27)) (justify left bottom))
   )
-  (text "ENCODER\n" (at 76.2 113.03 0)
+  (text "ENCODER\n" (at 101.6 100.33 0)
     (effects (font (size 1.27 1.27)) (justify left bottom))
   )

Commit message: 17:32
Connections:
- net GND: now reaches U?.4 (GND)
Other:
- note added: "Vcc is 5V"
- moved on the sheet: U?
Changed lines of the file:
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@@
 (kicad_sch (version 20230121) (generator eeschema)
   (paper "A4")
+  (wire (pts (xy 190.5 57.15) (xy 186.69 57.15))
+    (stroke (width 0) (type default))
+  )
+  (wire (pts (xy 186.69 57.15) (xy 186.69 59.69))
+    (stroke (width 0) (type default))
+  )
   (rectangle (start 83.82 40.64) (end 129.54 78.74)
     (stroke (width 0) (type default))
@@
     (fill (type none))
   )
-  (rectangle (start 166.37 40.64) (end 210.82 80.01)
+  (rectangle (start 166.37 40.64) (end 276.86 119.38)
     (stroke (width 0) (type default))
     (fill (type none))
@@
     (effects (font (size 1.27 1.27)) (justify left bottom))
   )
-  (symbol (lib_id "HC-SR04_ULTRASONIC_SENSOR:HC-SR04") (at 182.88 57.15 0) (unit 1)
+  (text "Vcc is 5V" (at 167.64 43.18 0)
+    (effects (font (size 1.27 1.27)) (justify left bottom))
+  )
+  (symbol (lib_id "power:GND") (at 186.69 59.69 0) (unit 1)
     (in_bom yes) (on_board yes) (dnp no) (fields_autoplaced)
-    (property "Reference" "U?" (at 194.31 57.785 0)
+    (property "Reference" "#PWR02" (at 186.69 66.04 0)
+      (effects (font (size 1.27 1.27)) hide)
+    )
+    (property "Value" "GND" (at 186.69 64.77 0)
+      (effects (font (size 1.27 1.27)))
+    )
+    (property "Footprint" "" (at 186.69 59.69 0)
+      (effects (font (size 1.27 1.27)) hide)
+    )
+    (property "Datasheet" "" (at 186.69 59.69 0)
+      (effects (font (size 1.27 1.27)) hide)
+    )
+    (pin "1")
+    (instances
+      (project "INDY THE TREASURE HUNTER"
+        (path "/b3b90d4c-73f4-4a78-9e6e-dd19a1913646/10de68d7-f5d9-4831-9d1b-771d16ee0d86"
+          (reference "#PWR02") (unit 1)
+        )
+      )
+    )
+  )
+  (symbol (lib_id "HC-SR04_ULTRASONIC_SENSOR:HC-SR04") (at 195.58 52.07 0) (unit 1)
+    (in_bom yes) (on_board yes) (dnp no) (fields_autoplaced)
+    (property "Reference" "U?" (at 207.01 52.705 0)
       (effects (font (size 1.27 1.27)) (justify left))
     )
-    (property "Value" "HC-SR04" (at 194.31 60.325 0)
+    (property "Value" "HC-SR04" (at 207.01 55.245 0)
       (effects (font (size 1.27 1.27)) (justify left))
     )
-    (property "Footprint" "XCVR_HC-SR04" (at 182.88 57.15 0)
+    (property "Footprint" "XCVR_HC-SR04" (at 195.58 52.07 0)
       (effects (font (size 1.27 1.27)) (justify bottom) hide)
     )
-    (property "Datasheet" "" (at 182.88 57.15 0)
+    (property "Datasheet" "" (at 195.58 52.07 0)
       (effects (font (size 1.27 1.27)) hide)
     )
-    (property "MF" "OSEPP Electronics" (at 182.88 57.15 0)
+    (property "MF" "OSEPP Electronics" (at 195.58 52.07 0)
       (effects (font (size 1.27 1.27)) (justify bottom) hide)
     )
-    (property "Description" "\nMultiple Function Sensor Development Tools Ultrasonic Sensor Module\n" (at 182.88 57.15 0)
+    (property "Description" "\nMultiple Function Sensor Development Tools Ultrasonic Sensor Module\n" (at 195.58 52.07 0)
       (effects (font (size 1.27 1.27)) (justify bottom) hide)
     )
-    (property "Package" "None" (at 182.88 57.15 0)
+    (property "Package" "None" (at 195.58 52.07 0)
       (effects (font (size 1.27 1.27)) (justify bottom) hide)
     )
-    (property "Price" "None" (at 182.88 57.15 0)
+    (property "Price" "None" (at 195.58 52.07 0)
       (effects (font (size 1.27 1.27)) (justify bottom) hide)
     )
-    (property "Check_prices" "https://www.snapeda.com/parts/HC-SR04/Applied+Avionics/view-part/?ref=eda" (at 182.88 57.15 0)
+    (property "Check_prices" "https://www.snapeda.com/parts/HC-SR04/Applied+Avionics/view-part/?ref=eda" (at 195.58 52.07 0)
       (effects (font (size 1.27 1.27)) (justify bottom) hide)
     )
-    (property "SnapEDA_Link" "https://www.snapeda.com/parts/HC-SR04/Applied+Avionics/view-part/?ref=snap" (at 182.88 57.15 0)
+    (property "SnapEDA_Link" "https://www.snapeda.com/parts/HC-SR04/Applied+Avionics/view-part/?ref=snap" (at 195.58 52.07 0)
       (effects (font (size 1.27 1.27)) (justify bottom) hide)
     )
-    (property "MP" "HC-SR04" (at 182.88 57.15 0)
+    (property "MP" "HC-SR04" (at 195.58 52.07 0)
       (effects (font (size 1.27 1.27)) (justify bottom) hide)
     )
-    (property "Purchase-URL" "https://pricing.snapeda.com/search?q=HC-SR04&ref=eda" (at 182.88 57.15 0)
+    (property "Purchase-URL" "https://pricing.snapeda.com/search?q=HC-SR04&ref=eda" (at 195.58 52.07 0)
       (effects (font (size 1.27 1.27)) (justify bottom) hide)
     )
-    (property "Availability" "In Stock" (at 182.88 57.15 0)
+    (property "Availability" "In Stock" (at 195.58 52.07 0)
       (effects (font (size 1.27 1.27)) (justify bottom) hide)
     )
-    (property "MANUFACTURER" "Osepp" (at 182.88 57.15 0)
+    (property "MANUFACTURER" "Osepp" (at 195.58 52.07 0)
       (effects (font (size 1.27 1.27)) (justify bottom) hide)
     )
@@
         )
         (path "/b3b90d4c-73f4-4a78-9e6e-dd19a1913646/10de68d7-f5d9-4831-9d1b-771d16ee0d86"
-          (reference "U?") (unit 1)
+          (reference "U1") (unit 1)
         )
       )
